File: pcb/steppersynth/steppersynth.kicad_sch (KiCad schematic)
At the start: 30 parts, among them J1 USB4105, J2 Conn_01x04_Pin, J3 LRS-350-24, SW1 SW_SPST, U1 ESP32-S3-WROOM-2, U2 TMC2209-LA, U3 LM3940IMPX-3.3/NOPB, U4 CD74HC4067M, U5 MCP6002-xMC

Commit message: update kicad stuff
Parts:
- removed C10, C11: 100nF, symbol Device:C_Small
- removed C7: 22nF, symbol Device:C_Small
- removed C8: 2.2µF, symbol Device:C_Small
- removed C9: 4.7µF, symbol Device:C_Small
- removed J2: Conn_01x04_Pin, symbol Connector:Conn_01x04_Pin
- removed R4: 0Ω, Resistor_SMD:R_0805_2012Metric, symbol Device:R_Small
- removed R7: 20kΩ, Resistor_SMD:R_0805_2012Metric, symbol Device:R_Small
- removed U2: TMC2209-LA, Package_DFN_QFN:VQFN-28-1EP_5x5mm_P0.5mm_EP3.7x3.7mm_ThermalVias, symbol Driver_Motor:TMC2209-LA
- removed U4: CD74HC4067M, Package_SO:SOIC-24W_7.5x15.4mm_P1.27mm, symbol 74xx:CD74HC4067M
- removed U5: MCP6002-xMC, Package_DFN_QFN:DFN-8-1EP_3x2mm_P0.5mm_EP1.75x1.45mm, symbol Amplifier_Operational:MCP6002-xMC
- added R2: 10kΩ, Resistor_SMD:R_0805_2012Metric, symbol Device:R_Small
- J2: renamed from J3; footprint (none) -> TerminalBlock_MetzConnect:TerminalBlock_MetzConnect_Type055_RT01502HDWU_1x02_P5.00mm_Horizontal
- TP1, TP2: footprint (none) -> MountingHole:MountingHole_3.2mm_M3_Pad
- renumbered C4 to C2, C6 to C3, C5 to C4, C2 to C5, C3 to C6, R3 to R1, R5 to R3, R6 to R4, R1 to R5, R2 to R6, U3 to U2
Connections:
- net VDD is gone; now on net +3.3V: U1.2 (3V3)
- net TMC1_DIR: now also U1.21 (IO13)
- net TMC1_PD_UART: now also U1.4 (IO4)
- net TMC1_STEP: now also U1.38 (IO2)
- net TMC3_STEP: now reaches U1.10 (IO17)
- net TMC3_DIR: now reaches U1.11 (IO18)
- net COM3: now reaches U1.12 (IO8)
- net RotB1: now reaches U1.15 (IO3)
- net RotB3: now reaches U1.16 (IO46)
- net S1: now reaches U1.17 (IO9)
- net S2: now reaches U1.18 (IO10)
- net S3: now reaches U1.19 (IO11)
- net RGB: now reaches U1.20 (IO12)
- net S0: now reaches U1.22 (IO14)
- net TMC3_PD_UART: now reaches U1.23 (IO21)
- net Switch1: now reaches U1.24 (IO47)
- net Switch2: now reaches U1.25 (IO48)
- net RotA3: now reaches U1.26 (IO45)
- net Switch3: now reaches U1.27 (IO0)
- net Switch3: now also R2.1
- net RotA2: now reaches U1.31 (IO38)
- net RotB2: now reaches U1.32 (MTCK/IO39)
- net TMC4_STEP: now reaches U1.33 (MTDO/IO40)
- net TMC4_DIR: now reaches U1.34 (MTDI/IO41)
- net TMC4_PD_UART: now reaches U1.35 (MTMS/IO42)
- net RotA1: now reaches U1.39 (IO1)
- net TMC2_STEP: now reaches U1.5 (IO5)
- net COM1: now reaches U1.6 (IO6)
- net COM2: now reaches U1.7 (IO7)
- net TMC2_DIR: now reaches U1.8 (IO15)
- net TMC2_PD_UART: now reaches U1.9 (IO16)
- net 24v renamed +24V
- net 3v3 renamed +3.3V
- net +3.3V: now also R2.2
- net 5v renamed +5V
- no-connect marks 6 -> 2
Other:
- added sheet Arpeggio Module (arp_mod.kicad_sch)
- added sheet Hall Effect Sensors (hall_sensors.kicad_sch)
- added sheet Motor Controllers (motor_controllers.kicad_sch)
- added sheet Sensor Mux (sensor_mux.kicad_sch)
- note removed: "TMC2209 Motor Controller"
- moved on the sheet: C2, C3, C4, D1, J1, J2, R1, R3, R4, R5, R6, SW1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

Commit message: dc-dc buck converter
Parts:
- added C81: 4.7μF, Capacitor_SMD:C_0805_2012Metric, symbol Device:C_Small
- added C82, C83: 0.1μF, Capacitor_SMD:C_0805_2012Metric, symbol Device:C_Small
- added J8: Conn_01x02_Pin, Connector_PinSocket_2.54mm:PinSocket_1x02_P2.54mm_Vertical, symbol Connector:Conn_01x02_Pin
- added J9: Conn_01x02_Socket, Connector_PinSocket_2.54mm:PinSocket_1x02_P2.54mm_Vertical, symbol Connector:Conn_01x02_Socket
- added R26: 10kΩ, Resistor_SMD:R_0805_2012Metric, symbol Device:R_Small
- added R27: 100kΩ, Resistor_SMD:R_0805_2012Metric, symbol Device:R_Small
- added U49: TPS2115APW, 2_udu_lib:PW8, symbol 3_udu_lib:TPS2115APW
Connections:
- net +24V: now also J9.1 (Pin_1)
- net +5V: now also C81.1, U49.7 (OUT); no longer D1.1 (K)
- net GND: now also C81.2, C82.1, C83.2, J8.2 (Pin_2), J9.2 (Pin_2), R27.1, U49.2 (D0), U49.5 (GND)
- new net: R26.2, R27.2, U49.3 (D1)
- new net IN1: C82.2, J8.1 (Pin_1), R26.1, U49.8 (IN1)
- new net IN2: C83.1, D1.1 (K), U49.6 (IN2)
- no-connect marks 2 -> 4
Other:
- note added: "Autoswitching power mux"
- note added: "External 24V -> 5v DC-DC Buck Converter Module"
- note added: "module here"
- moved on the sheet: D1, J1, R5, R6
