File: pcb/steppersynth/motor_controllers.kicad_sch (KiCad schematic)
At the start: 32 parts, among them J3 Conn_01x04_Pin, J4 Conn_01x04_Pin, J5 Conn_01x04_Pin, J6 Conn_01x04_Pin, U3 TMC2209-LA, U4 TMC2209-LA, U5 TMC2209-LA, U6 TMC2209-LA

Commit message: fix tmc motor stuff + more
Parts:
- removed C10, C9: 100nF, Capacitor_SMD:C_0805_2012Metric, symbol Device:C_Small
- removed C19: 2.2µF, Capacitor_SMD:C_0805_2012Metric, symbol Device:C_Small
- removed C25: 22nF, Capacitor_SMD:C_0805_2012Metric, symbol Device:C_Small
- added C10, C19, C25, C9: 150µF, Capacitor_THT:C_Radial_D12.5mm_H25.0mm_P5.00mm, symbol Device:C_Polarized_Small
- added C77: 100nF, Capacitor_SMD:C_0805_2012Metric, symbol Device:C_Small
- added C78: 2.2µF, Capacitor_SMD:C_0805_2012Metric, symbol Device:C_Small
- added C79: 22nF, Capacitor_SMD:C_0805_2012Metric, symbol Device:C_Small
- added C80: 4.7µF, Capacitor_SMD:C_0805_2012Metric, symbol Device:C_Small
- added R22, R24: 20kΩ, Resistor_SMD:R_0805_2012Metric, symbol Device:R_Small
- added R23, R25: 1kΩ, Resistor_SMD:R_0805_2012Metric, symbol Device:R_Small
- C12: value 2.2µF -> 100nF
- C14, C20: value 22nF -> 100nF
- C16: value 4.7µF -> 2.2µF
- C17, C23: value 100nF -> 22nF
- C18: value 100nF -> 4.7µF
- C21, C26: value 4.7µF -> 100nF
- C22: value 100nF -> 2.2µF
- C24: value 2.2µF -> 4.7µF
- R10, R8: value 20kΩ -> 1kΩ
Connections:
- net +24V: now also C12.1, C14.1, C20.1, C21.1, C26.1, C8.1, C10.1, C19.1, C25.1, C77.1, C9.1; no longer C17.1, C22.1
- net GND: now also C18.2, C20.2, C22.2, C8.2, C10.2, C19.2, C25.2, C78.2, C80.2, C9.2, R22.1, R24.1; no longer C18.1, C21.2, C23.1, C8.1, R10.1, R8.1
- net TMC1_PD_UART: now also R8.1; no longer U3.14 (~{PD}/UART)
- net TMC2_PD_UART: now also R10.1; no longer U4.14 (~{PD}/UART)
- net TMC3_PD_UART: now also R23.1; no longer U5.14 (~{PD}/UART)
- net TMC4_PD_UART: now also R25.1; no longer U6.14 (~{PD}/UART)
- net at C7.2, U3.6 (VCP): no longer C8.2
- net at U4.6 (VCP): now also C14.2
- net at C16.1, U4.8 (5VOUT): now also C18.1; no longer C12.1
- net at U6.2 (~{EN}): now also R24.2; no longer R10.2
- net at U5.8 (5VOUT): now also C22.1, C24.1; no longer C21.1
- net at R9.2: now also U4.2 (~{EN}); no longer U5.2 (~{EN})
- net at U5.4 (CPO): now also C23.1; no longer C20.1
- net at U5.5 (CPI): now also C23.2; no longer C20.2
- net at U6.4 (CPO): now also C79.1
- net at U6.5 (CPI): now also C79.2
- net at R8.2: now also U3.14 (~{PD}/UART); no longer U4.2 (~{EN})
- net at U4.4 (CPO): now also C17.1; no longer C14.1
- net at U4.5 (CPI): now also C17.2; no longer C14.2
- new net: R23.2, U5.14 (~{PD}/UART)
- new net: C77.2, U6.6 (VCP)
- new net: C78.1, C80.1, U6.8 (5VOUT)
- new net: R10.2, U4.14 (~{PD}/UART)
- new net: R25.2, U6.14 (~{PD}/UART)
- new net: R22.2, U5.2 (~{EN})
- new net: C21.2, U5.6 (VCP)
Other:
- moved on the sheet: C8

Commit message: position everything in the pcb
Parts:
- C10, C19, C25, C9: footprint Capacitor_THT:C_Radial_D12.5mm_H25.0mm_P5.00mm -> Capacitor_THT:C_Radial_D10.0mm_H12.5mm_P5.00mm
Changed lines of the file:
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@@
 			)
 		)
-		(property "Footprint" "Capacitor_THT:C_Radial_D12.5mm_H25.0mm_P5.00mm"
+		(property "Footprint" "Capacitor_THT:C_Radial_D10.0mm_H12.5mm_P5.00mm"
 			(at 201.93 30.48 0)
 			(effects
@@
 			)
 		)
-		(property "Footprint" "Capacitor_THT:C_Radial_D12.5mm_H25.0mm_P5.00mm"
+		(property "Footprint" "Capacitor_THT:C_Radial_D10.0mm_H12.5mm_P5.00mm"
 			(at 26.67 30.48 0)
 			(effects
@@
 			)
 		)
-		(property "Footprint" "Capacitor_THT:C_Radial_D12.5mm_H25.0mm_P5.00mm"
+		(property "Footprint" "Capacitor_THT:C_Radial_D10.0mm_H12.5mm_P5.00mm"
 			(at 114.3 30.48 0)
 			(effects
@@
 			)
 		)
-		(property "Footprint" "Capacitor_THT:C_Radial_D12.5mm_H25.0mm_P5.00mm"
+		(property "Footprint" "Capacitor_THT:C_Radial_D10.0mm_H12.5mm_P5.00mm"
 			(at 26.67 110.49 0)
 			(effects

Commit message: finish tracing everything
Connections:
- net at J6.2 (Pin_2): now also U6.26 (OB1); no longer U6.21 (OA2)
- net at J6.3 (Pin_3): now also U6.21 (OA2); no longer U6.26 (OB1)
- net at U4.21 (OA2): now also J4.3 (Pin_3); no longer J4.2 (Pin_2)
- net at U4.26 (OB1): now also J4.2 (Pin_2); no longer J4.3 (Pin_3)
- net at U3.21 (OA2): now also J3.3 (Pin_3); no longer J3.2 (Pin_2)
- net at U3.26 (OB1): now also J3.2 (Pin_2); no longer J3.3 (Pin_3)
- net at J5.2 (Pin_2): now also U5.26 (OB1); no longer U5.21 (OA2)
- net at J5.3 (Pin_3): now also U5.21 (OA2); no longer U5.26 (OB1)
