File: pcb/steppersynth/steppersynth.kicad_pcb (KiCad board)
At the start: 2 copper layers, 0 parts

Commit message: position everything in the pcb
Parts:
- added C1: 1uF, Capacitor_SMD:C_0805_2012Metric, B.Cu at (155.1, 60.9)
- added C10: 150µF, Capacitor_THT:C_Radial_D10.0mm_H12.5mm_P5.00mm, B.Cu at (21.1, 102.8)
- added C11: 2.2µF, Capacitor_SMD:C_0805_2012Metric, B.Cu at (50.6, 89.7)
- added C12: 100nF, Capacitor_SMD:C_0805_2012Metric, B.Cu at (44.9, 93.0)
- added C13: 22nF, Capacitor_SMD:C_0805_2012Metric, B.Cu at (53.5, 86.1)
- added C14: 100nF, Capacitor_SMD:C_0805_2012Metric, B.Cu at (54.2, 97.8)
- added C15: 4.7µF, Capacitor_SMD:C_0805_2012Metric, B.Cu at (47.0, 89.8)
- added C16: 2.2µF, Capacitor_SMD:C_0805_2012Metric, B.Cu at (46.9, 98.7)
- added C17: 22nF, Capacitor_SMD:C_0805_2012Metric, B.Cu at (53.4, 95.0)
- added C18: 4.7µF, Capacitor_SMD:C_0805_2012Metric, B.Cu at (50.6, 98.8)
- added C19: 150µF, Capacitor_THT:C_Radial_D10.0mm_H12.5mm_P5.00mm, B.Cu at (37.4, 94.5)
- added C2: 10μF, Capacitor_SMD:C_0805_2012Metric, B.Cu at (154.9, 56.6)
- added C20: 100nF, Capacitor_SMD:C_0805_2012Metric, B.Cu at (57.2, 84.2)
- added C21: 100nF, Capacitor_SMD:C_0805_2012Metric, B.Cu at (66.6, 89.0)
- added C22: 2.2µF, Capacitor_SMD:C_0805_2012Metric, B.Cu at (59.3, 89.9)
- added C23: 22nF, Capacitor_SMD:C_0805_2012Metric, B.Cu at (65.8, 86.1)
- added C24: 4.7µF, Capacitor_SMD:C_0805_2012Metric, B.Cu at (62.9, 89.9)
- added C25: 150µF, Capacitor_THT:C_Radial_D10.0mm_H12.5mm_P5.00mm, B.Cu at (21.1, 113.8)
- added C26: 100nF, Capacitor_SMD:C_0805_2012Metric, B.Cu at (57.6, 93.3)
- added C27: 0.01µF, Capacitor_SMD:C_0805_2012Metric, B.Cu at (24.6, 123.6)
- added C28: 0.01µF, Capacitor_SMD:C_0805_2012Metric, B.Cu at (43.7, 123.6)
- added C29: 0.01µF, Capacitor_SMD:C_0805_2012Metric, B.Cu at (62.8, 123.6)
- added C3: 0.1μF, Capacitor_SMD:C_0805_2012Metric, B.Cu at (157.9, 61.8)
- added C30: 0.01µF, Capacitor_SMD:C_0805_2012Metric, B.Cu at (81.8, 123.6)
- added C31: 0.01µF, Capacitor_SMD:C_0805_2012Metric, B.Cu at (100.9, 123.6)
- added C32: 0.01µF, Capacitor_SMD:C_0805_2012Metric, B.Cu at (119.9, 123.6)
- added C33: 0.01µF, Capacitor_SMD:C_0805_2012Metric, B.Cu at (139.0, 123.6)
- added C34: 0.01µF, Capacitor_SMD:C_0805_2012Metric, B.Cu at (34.0, 104.6)
- added C35: 0.01µF, Capacitor_SMD:C_0805_2012Metric, B.Cu at (53.2, 104.7)
- added C36: 0.01µF, Capacitor_SMD:C_0805_2012Metric, B.Cu at (91.3, 104.7)
- added C37: 0.01µF, Capacitor_SMD:C_0805_2012Metric, B.Cu at (110.5, 104.7)
- added C38: 0.01µF, Capacitor_SMD:C_0805_2012Metric, B.Cu at (129.2, 104.7)
- added C39: 0.01µF, Capacitor_SMD:C_0805_2012Metric, B.Cu at (158.0, 123.6)
- added C4: 0.1μF, Capacitor_SMD:C_0805_2012Metric, B.Cu at (154.9, 58.7)
- added C40: 0.01µF, Capacitor_SMD:C_0805_2012Metric, B.Cu at (177.1, 123.6)
- added C41: 0.01µF, Capacitor_SMD:C_0805_2012Metric, B.Cu at (196.1, 123.6)
- added C42: 0.01µF, Capacitor_SMD:C_0805_2012Metric, B.Cu at (215.2, 123.6)
- added C43: 0.01µF, Capacitor_SMD:C_0805_2012Metric, B.Cu at (234.2, 123.6)
- added C44: 0.01µF, Capacitor_SMD:C_0805_2012Metric, B.Cu at (253.3, 123.6)
- added C45: 0.01µF, Capacitor_SMD:C_0805_2012Metric, B.Cu at (272.4, 123.6)
- added C46: 0.01µF, Capacitor_SMD:C_0805_2012Metric, B.Cu at (167.4, 104.6)
- added C47: 0.01µF, Capacitor_SMD:C_0805_2012Metric, B.Cu at (186.7, 104.7)
- added C48: 0.01µF, Capacitor_SMD:C_0805_2012Metric, B.Cu at (224.7, 104.8)
- added C49: 0.01µF, Capacitor_SMD:C_0805_2012Metric, B.Cu at (243.8, 104.7)
- added C5: 0.47μF, Capacitor_SMD:C_0805_2012Metric, B.Cu at (260.0, 74.0)
- added C50: 0.01µF, Capacitor_SMD:C_0805_2012Metric, B.Cu at (262.6, 104.8)
- added C51: 0.01µF, Capacitor_SMD:C_0805_2012Metric, B.Cu at (158.1, 80.8)
- added C52: 0.01µF, Capacitor_SMD:C_0805_2012Metric, B.Cu at (177.1, 80.8)
- added C53: 0.01µF, Capacitor_SMD:C_0805_2012Metric, B.Cu at (196.1, 80.8)
- added C54: 0.01µF, Capacitor_SMD:C_0805_2012Metric, B.Cu at (215.1, 80.8)
- added C55: 0.01µF, Capacitor_SMD:C_0805_2012Metric, B.Cu at (234.1, 80.8)
- added C56: 0.01µF, Capacitor_SMD:C_0805_2012Metric, B.Cu at (253.1, 80.8)
- added C57: 0.01µF, Capacitor_SMD:C_0805_2012Metric, B.Cu at (272.1, 80.8)
- added C58: 0.01µF, Capacitor_SMD:C_0805_2012Metric, B.Cu at (167.6, 61.7)
- added C59: 0.01µF, Capacitor_SMD:C_0805_2012Metric, B.Cu at (186.6, 61.8)
- added C6: 47μF, Capacitor_SMD:C_0805_2012Metric, B.Cu at (260.0, 70.5)
- added C60: 0.01µF, Capacitor_SMD:C_0805_2012Metric, B.Cu at (224.7, 61.7)
- added C61: 0.01µF, Capacitor_SMD:C_0805_2012Metric, B.Cu at (243.6, 61.6)
- added C62: 0.01µF, Capacitor_SMD:C_0805_2012Metric, B.Cu at (262.9, 61.7)
- added C63: 100nF, Capacitor_SMD:C_0805_2012Metric, B.Cu at (64.3, 102.8)
- added C64: 100nF, Capacitor_SMD:C_0805_2012Metric, B.Cu at (196.9, 59.9)
- added C65: 100nF, Capacitor_SMD:C_0805_2012Metric, B.Cu at (64.3, 112.0)
- added C66: 100nF, Capacitor_SMD:C_0805_2012Metric, B.Cu at (197.1, 69.2)
- added C67: 100nF, Capacitor_SMD:C_0805_2012Metric, B.Cu at (197.7, 102.4)
- added C68: 100nF, Capacitor_SMD:C_0805_2012Metric, B.Cu at (197.6, 111.5)
- added C69: 100nF, Capacitor_SMD:C_0805_2012Metric, B.Cu at (35.1, 78.2)
- added C7: 100nF, Capacitor_SMD:C_0805_2012Metric, B.Cu at (54.2, 88.8)
- added C70: 100nF, Capacitor_SMD:C_0805_2012Metric, B.Cu at (47.9, 78.2)
- added C71: 100nF, Capacitor_SMD:C_0805_2012Metric, B.Cu at (60.6, 78.2)
- added C72: 100nF, Capacitor_SMD:C_0805_2012Metric, B.Cu at (73.4, 78.2)
- added C73: 100nF, Capacitor_SMD:C_0805_2012Metric, B.Cu at (86.1, 78.2)
- added C74: 100nF, Capacitor_SMD:C_0805_2012Metric, B.Cu at (98.8, 78.2)
- added C75: 100nF, Capacitor_SMD:C_0805_2012Metric, B.Cu at (111.6, 78.2)
- added C76: 100nF, Capacitor_SMD:C_0805_2012Metric, B.Cu at (124.3, 78.2)
- added C77: 100nF, Capacitor_SMD:C_0805_2012Metric, B.Cu at (66.7, 98.1)
- added C78: 2.2µF, Capacitor_SMD:C_0805_2012Metric, B.Cu at (59.5, 99.1)
- added C79: 22nF, Capacitor_SMD:C_0805_2012Metric, B.Cu at (66.0, 95.3)
- added C8: 100nF, Capacitor_SMD:C_0805_2012Metric, B.Cu at (44.8, 84.0)
- added C80: 4.7µF, Capacitor_SMD:C_0805_2012Metric, B.Cu at (63.1, 99.1)
- added C9: 150µF, Capacitor_THT:C_Radial_D10.0mm_H12.5mm_P5.00mm, B.Cu at (37.4, 83.4)
- added D1: SS14, Diode_SMD:D_SMA, B.Cu at (274.7, 71.6)
- added D2: WS2812B, LED_SMD:LED_WS2812B_PLCC4_5.0x5.0mm_P3.2mm, F.Cu at (39.8, 79.2)
- added D3: WS2812B, LED_SMD:LED_WS2812B_PLCC4_5.0x5.0mm_P3.2mm, F.Cu at (52.5, 79.2)
- added D4: WS2812B, LED_SMD:LED_WS2812B_PLCC4_5.0x5.0mm_P3.2mm, F.Cu at (65.2, 79.2)
- added D5: WS2812B, LED_SMD:LED_WS2812B_PLCC4_5.0x5.0mm_P3.2mm, F.Cu at (77.9, 79.2)
- added D6: WS2812B, LED_SMD:LED_WS2812B_PLCC4_5.0x5.0mm_P3.2mm, F.Cu at (90.6, 79.2)
- added D7: WS2812B, LED_SMD:LED_WS2812B_PLCC4_5.0x5.0mm_P3.2mm, F.Cu at (103.3, 79.2)
- added D8: WS2812B, LED_SMD:LED_WS2812B_PLCC4_5.0x5.0mm_P3.2mm, F.Cu at (116.0, 79.2)
- added D9: WS2812B, LED_SMD:LED_WS2812B_PLCC4_5.0x5.0mm_P3.2mm, F.Cu at (128.8, 79.2)
- added J1: USB4105, Connector_USB:USB_C_Receptacle_GCT_USB4105-xx-A_16P_TopMnt_Horizontal, B.Cu at (277.9, 64.3)
- added J2: LRS-350-24, TerminalBlock_MetzConnect:TerminalBlock_MetzConnect_Type055_RT01502HDWU_1x02_P5.00mm_Horizontal, B.Cu at (18.8, 95.4)
- added J3: Conn_01x04_Pin, Connector_PinHeader_2.54mm:PinHeader_1x04_P2.54mm_Vertical, B.Cu at (34.6, 60.6)
- added J4: Conn_01x04_Pin, Connector_PinHeader_2.54mm:PinHeader_1x04_P2.54mm_Vertical, B.Cu at (56.8, 60.7)
- added J5: Conn_01x04_Pin, Connector_PinHeader_2.54mm:PinHeader_1x04_P2.54mm_Vertical, B.Cu at (28.0, 73.9)
- added J6: Conn_01x04_Pin, Connector_PinHeader_2.54mm:PinHeader_1x04_P2.54mm_Vertical, B.Cu at (48.6, 73.7)
- added R1: 10kΩ, Resistor_SMD:R_0805_2012Metric, B.Cu at (155.0, 62.9)
- added R10: 1kΩ, Resistor_SMD:R_0805_2012Metric, B.Cu at (154.8, 67.0)
- added R11: 10kΩ, Resistor_SMD:R_0805_2012Metric, B.Cu at (78.1, 115.7)
- added R12: 10kΩ, Resistor_SMD:R_0805_2012Metric, B.Cu at (210.7, 72.6)
- added R13: 10kΩ, Resistor_SMD:R_0805_2012Metric, B.Cu at (211.4, 115.2)
- added R14: 220Ω, Resistor_SMD:R_0805_2012Metric, B.Cu at (44.4, 80.3)
- added R15: 220Ω, Resistor_SMD:R_0805_2012Metric, B.Cu at (57.1, 80.3)
- added R16: 220Ω, Resistor_SMD:R_0805_2012Metric, B.Cu at (69.8, 80.3)
- added R17: 220Ω, Resistor_SMD:R_0805_2012Metric, B.Cu at (82.5, 80.3)
- added R18: 220Ω, Resistor_SMD:R_0805_2012Metric, B.Cu at (95.2, 80.3)
- added R19: 220Ω, Resistor_SMD:R_0805_2012Metric, B.Cu at (107.9, 80.3)
- added R2: 10kΩ, Resistor_SMD:R_0805_2012Metric, B.Cu at (122.5, 72.6)
- added R20: 220Ω, Resistor_SMD:R_0805_2012Metric, B.Cu at (120.7, 80.3)
- added R21: 220Ω, Resistor_SMD:R_0805_2012Metric, B.Cu at (133.4, 80.3)
- added R22: 20kΩ, Resistor_SMD:R_0805_2012Metric, B.Cu at (66.5, 83.4)
- added R23: 1kΩ, Resistor_SMD:R_0805_2012Metric, B.Cu at (135.8, 80.3)
- added R24: 20kΩ, Resistor_SMD:R_0805_2012Metric, B.Cu at (66.7, 92.5)
- added R25: 1kΩ, Resistor_SMD:R_0805_2012Metric, B.Cu at (122.0, 62.4)
- added R3: 0Ω, Resistor_SMD:R_0805_2012Metric, B.Cu at (155.4, 71.5)
- added R4: 0Ω, Resistor_SMD:R_0805_2012Metric, B.Cu at (155.4, 73.6)
- added R5: 5.1kΩ, Resistor_SMD:R_0805_2012Metric, B.Cu at (272.1, 62.3)
- added R6: 5.1kΩ, Resistor_SMD:R_0805_2012Metric, B.Cu at (272.1, 66.8)
- added R7: 20kΩ, Resistor_SMD:R_0805_2012Metric, B.Cu at (54.2, 83.3)
- added R8: 1kΩ, Resistor_SMD:R_0805_2012Metric, B.Cu at (154.9, 65.0)
- added R9: 20kΩ, Resistor_SMD:R_0805_2012Metric, B.Cu at (54.1, 92.2)
- added REF**: SW_Cherry_MX_1.00u_PCB, Button_Switch_Keyboard:SW_Cherry_MX_1.00u_PCB, F.Cu at (131.8, 102.3)
- added REF**: SW_Cherry_MX_1.00u_PCB, Button_Switch_Keyboard:SW_Cherry_MX_1.00u_PCB, F.Cu at (236.6, 121.3)
- added REF**: SW_Cherry_MX_1.00u_PCB, Button_Switch_Keyboard:SW_Cherry_MX_1.00u_PCB, F.Cu at (36.6, 102.3)
- added REF**: SW_Cherry_MX_1.00u_PCB, Button_Switch_Keyboard:SW_Cherry_MX_1.00u_PCB, F.Cu at (55.6, 102.3)
- added REF**: SW_Cherry_MX_1.00u_PCB, Button_Switch_Keyboard:SW_Cherry_MX_1.00u_PCB, F.Cu at (46.1, 121.3)
- added REF**: SW_Cherry_MX_1.00u_PCB, Button_Switch_Keyboard:SW_Cherry_MX_1.00u_PCB, F.Cu at (112.8, 102.3)
- added REF**: SW_Cherry_MX_1.00u_PCB, Button_Switch_Keyboard:SW_Cherry_MX_1.00u_PCB, F.Cu at (227.1, 59.5)
- added REF**: SW_Cherry_MX_1.00u_PCB, Button_Switch_Keyboard:SW_Cherry_MX_1.00u_PCB, F.Cu at (198.5, 121.3)
- added REF**: SW_Cherry_MX_1.00u_PCB, Button_Switch_Keyboard:SW_Cherry_MX_1.00u_PCB, F.Cu at (160.4, 78.5)
- added REF**: SW_Cherry_MX_1.00u_PCB, Button_Switch_Keyboard:SW_Cherry_MX_1.00u_PCB, F.Cu at (65.2, 121.3)
- added REF**: SW_Cherry_MX_1.00u_PCB, Button_Switch_Keyboard:SW_Cherry_MX_1.00u_PCB, F.Cu at (179.5, 121.3)
- added REF**: SW_Cherry_MX_1.00u_PCB, Button_Switch_Keyboard:SW_Cherry_MX_1.00u_PCB, F.Cu at (84.2, 121.3)
- added REF**: SW_Cherry_MX_1.00u_PCB, Button_Switch_Keyboard:SW_Cherry_MX_1.00u_PCB, F.Cu at (189.0, 102.3)
- added REF**: SW_Cherry_MX_1.00u_PCB, Button_Switch_Keyboard:SW_Cherry_MX_1.00u_PCB, F.Cu at (274.7, 121.3)
- added REF**: SW_Cherry_MX_1.00u_PCB, Button_Switch_Keyboard:SW_Cherry_MX_1.00u_PCB, F.Cu at (103.3, 121.3)
- added REF**: SW_Cherry_MX_1.00u_PCB, Button_Switch_Keyboard:SW_Cherry_MX_1.00u_PCB, F.Cu at (265.2, 102.3)
- added REF**: SW_Cherry_MX_1.00u_PCB, Button_Switch_Keyboard:SW_Cherry_MX_1.00u_PCB, F.Cu at (169.9, 102.3)
- added REF**: SW_Cherry_MX_1.00u_PCB, Button_Switch_Keyboard:SW_Cherry_MX_1.00u_PCB, F.Cu at (217.6, 78.5)
- added REF**: SW_Cherry_MX_1.00u_PCB, Button_Switch_Keyboard:SW_Cherry_MX_1.00u_PCB, F.Cu at (217.6, 121.3)
- added REF**: SW_Cherry_MX_1.00u_PCB, Button_Switch_Keyboard:SW_Cherry_MX_1.00u_PCB, F.Cu at (255.7, 78.5)
- added REF**: SW_Cherry_MX_1.00u_PCB, Button_Switch_Keyboard:SW_Cherry_MX_1.00u_PCB, F.Cu at (160.4, 121.3)
- added REF**: SW_Cherry_MX_1.00u_PCB, Button_Switch_Keyboard:SW_Cherry_MX_1.00u_PCB, F.Cu at (189.0, 59.5)
- added REF**: SW_Cherry_MX_1.00u_PCB, Button_Switch_Keyboard:SW_Cherry_MX_1.00u_PCB, F.Cu at (227.1, 102.3)
- added REF**: SW_Cherry_MX_1.00u_PCB, Button_Switch_Keyboard:SW_Cherry_MX_1.00u_PCB, F.Cu at (246.1, 102.3)
- added REF**: SW_Cherry_MX_1.00u_PCB, Button_Switch_Keyboard:SW_Cherry_MX_1.00u_PCB, F.Cu at (255.7, 121.3)
- added REF**: SW_Cherry_MX_1.00u_PCB, Button_Switch_Keyboard:SW_Cherry_MX_1.00u_PCB, F.Cu at (141.4, 121.3)
- added REF**: SW_Cherry_MX_1.00u_PCB, Button_Switch_Keyboard:SW_Cherry_MX_1.00u_PCB, F.Cu at (122.3, 121.3)
- added REF**: SW_Cherry_MX_1.00u_PCB, Button_Switch_Keyboard:SW_Cherry_MX_1.00u_PCB, F.Cu at (265.2, 59.5)
- added REF**: SW_Cherry_MX_1.00u_PCB, Button_Switch_Keyboard:SW_Cherry_MX_1.00u_PCB, F.Cu at (274.7, 78.5)
- added REF**: SW_Cherry_MX_1.00u_PCB, Button_Switch_Keyboard:SW_Cherry_MX_1.00u_PCB, F.Cu at (27.1, 59.5)
- added REF**: SW_Cherry_MX_1.00u_PCB, Button_Switch_Keyboard:SW_Cherry_MX_1.00u_PCB, F.Cu at (198.5, 78.5)
- added REF**: SW_Cherry_MX_1.00u_PCB, Button_Switch_Keyboard:SW_Cherry_MX_1.00u_PCB, F.Cu at (27.1, 78.5)
- added REF**: SW_Cherry_MX_1.00u_PCB, Button_Switch_Keyboard:SW_Cherry_MX_1.00u_PCB, F.Cu at (246.1, 59.5)
- added REF**: SW_Cherry_MX_1.00u_PCB, Button_Switch_Keyboard:SW_Cherry_MX_1.00u_PCB, F.Cu at (179.5, 78.5)
- added REF**: SW_Cherry_MX_1.00u_PCB, Button_Switch_Keyboard:SW_Cherry_MX_1.00u_PCB, F.Cu at (169.9, 59.5)
- added REF**: SW_Cherry_MX_1.00u_PCB, Button_Switch_Keyboard:SW_Cherry_MX_1.00u_PCB, F.Cu at (236.6, 78.5)
- added REF**: SW_Cherry_MX_1.00u_PCB, Button_Switch_Keyboard:SW_Cherry_MX_1.00u_PCB, F.Cu at (93.7, 102.3)
- added REF**: SW_Cherry_MX_1.00u_PCB, Button_Switch_Keyboard:SW_Cherry_MX_1.00u_PCB, F.Cu at (27.1, 121.3)
- added SW1: SW_SPST, Button_Switch_THT:SW_PUSH_6mm, F.Cu at (108.2, 62.8)
- added SW2: RotaryEncoder_Switch, Rotary_Encoder:RotaryEncoder_Alps_EC11E-Switch_Vertical_H20mm, F.Cu at (38.2, 62.5)
- added SW3: SW_Push_45deg, EasyEDA:TH_L10.9-W5.9-CPG151101S11, B.Cu at (23.9, 60.7)
- added SW4: SW_Push_45deg, EasyEDA:TH_L10.9-W5.9-CPG151101S11, B.Cu at (23.8, 79.8)
- added SW5: RotaryEncoder_Switch, Rotary_Encoder:RotaryEncoder_Alps_EC11E-Switch_Vertical_H20mm, F.Cu at (61.0, 62.5)
- added SW6: RotaryEncoder_Switch, Rotary_Encoder:RotaryEncoder_Alps_EC11E-Switch_Vertical_H20mm, F.Cu at (83.8, 62.5)
- added TP1 TX: TestPoint, MountingHole:MountingHole_3.2mm_M3_Pad, F.Cu at (277.0, 99.2)
- added TP2 RX: TestPoint, MountingHole:MountingHole_3.2mm_M3_Pad, F.Cu at (277.0, 109.5)
- added U1: ESP32-S3-WROOM-2, RF_Module:ESP32-S3-WROOM-2, B.Cu at (138.6, 61.5)
- added U10: DRV5055A3xDBZxQ1, Package_TO_SOT_SMD:SOT-23, B.Cu at (81.8, 126.4)
- added U11: DRV5055A3xDBZxQ1, Package_TO_SOT_SMD:SOT-23, B.Cu at (100.8, 126.4)
- added U12: DRV5055A3xDBZxQ1, Package_TO_SOT_SMD:SOT-23, B.Cu at (119.9, 126.4)
- added U13: DRV5055A3xDBZxQ1, Package_TO_SOT_SMD:SOT-23, B.Cu at (138.9, 126.4)
- added U14: DRV5055A3xDBZxQ1, Package_TO_SOT_SMD:SOT-23, B.Cu at (34.0, 107.5)
- added U15: DRV5055A3xDBZxQ1, Package_TO_SOT_SMD:SOT-23, B.Cu at (53.3, 107.5)
- added U16: DRV5055A3xDBZxQ1, Package_TO_SOT_SMD:SOT-23, B.Cu at (91.4, 107.5)
- added U17: DRV5055A3xDBZxQ1, Package_TO_SOT_SMD:SOT-23, B.Cu at (110.4, 107.5)
- added U18: DRV5055A3xDBZxQ1, Package_TO_SOT_SMD:SOT-23, B.Cu at (129.2, 107.5)
- added U19: DRV5055A3xDBZxQ1, Package_TO_SOT_SMD:SOT-23, B.Cu at (158.0, 126.4)
- added U2: LM3940IMPX-3.3/NOPB, EasyEDA:SOT-223-4_L6.5-W3.5-P2.30-LS7.0-BR, B.Cu at (265.5, 72.2)
- added U20: DRV5055A3xDBZxQ1, Package_TO_SOT_SMD:SOT-23, B.Cu at (177.0, 126.4)
- added U21: DRV5055A3xDBZxQ1, Package_TO_SOT_SMD:SOT-23, B.Cu at (196.1, 126.4)
- added U22: DRV5055A3xDBZxQ1, Package_TO_SOT_SMD:SOT-23, B.Cu at (215.1, 126.4)
- added U23: DRV5055A3xDBZxQ1, Package_TO_SOT_SMD:SOT-23, B.Cu at (234.2, 126.4)
- added U24: DRV5055A3xDBZxQ1, Package_TO_SOT_SMD:SOT-23, B.Cu at (253.2, 126.4)
- added U25: DRV5055A3xDBZxQ1, Package_TO_SOT_SMD:SOT-23, B.Cu at (272.3, 126.4)
- added U26: DRV5055A3xDBZxQ1, Package_TO_SOT_SMD:SOT-23, B.Cu at (167.4, 107.5)
- added U27: DRV5055A3xDBZxQ1, Package_TO_SOT_SMD:SOT-23, B.Cu at (186.6, 107.5)
- added U28: DRV5055A3xDBZxQ1, Package_TO_SOT_SMD:SOT-23, B.Cu at (224.6, 107.5)
- added U29: DRV5055A3xDBZxQ1, Package_TO_SOT_SMD:SOT-23, B.Cu at (243.8, 107.5)
- added U3: TMC2209-LA, Package_DFN_QFN:VQFN-28-1EP_5x5mm_P0.5mm_EP3.7x3.7mm_ThermalVias, B.Cu at (49.0, 85.4)
- added U30: DRV5055A3xDBZxQ1, Package_TO_SOT_SMD:SOT-23, B.Cu at (262.6, 107.5)
- added U31: DRV5055A3xDBZxQ1, Package_TO_SOT_SMD:SOT-23, B.Cu at (158.0, 83.5)
- added U32: DRV5055A3xDBZxQ1, Package_TO_SOT_SMD:SOT-23, B.Cu at (177.0, 83.5)
- added U33: DRV5055A3xDBZxQ1, Package_TO_SOT_SMD:SOT-23, B.Cu at (196.1, 83.5)
- added U34: DRV5055A3xDBZxQ1, Package_TO_SOT_SMD:SOT-23, B.Cu at (215.1, 83.5)
- added U35: DRV5055A3xDBZxQ1, Package_TO_SOT_SMD:SOT-23, B.Cu at (234.2, 83.5)
- added U36: DRV5055A3xDBZxQ1, Package_TO_SOT_SMD:SOT-23, B.Cu at (253.2, 83.5)
- added U37: DRV5055A3xDBZxQ1, Package_TO_SOT_SMD:SOT-23, B.Cu at (272.2, 83.5)
- added U38: DRV5055A3xDBZxQ1, Package_TO_SOT_SMD:SOT-23, B.Cu at (167.5, 64.5)
- added U39: DRV5055A3xDBZxQ1, Package_TO_SOT_SMD:SOT-23, B.Cu at (186.5, 64.5)
- added U4: TMC2209-LA, Package_DFN_QFN:VQFN-28-1EP_5x5mm_P0.5mm_EP3.7x3.7mm_ThermalVias, B.Cu at (49.2, 94.4)
- added U40: DRV5055A3xDBZxQ1, Package_TO_SOT_SMD:SOT-23, B.Cu at (224.6, 64.4)
- added U41: DRV5055A3xDBZxQ1, Package_TO_SOT_SMD:SOT-23, B.Cu at (243.6, 64.4)
- added U42: DRV5055A3xDBZxQ1, Package_TO_SOT_SMD:SOT-23, B.Cu at (262.8, 64.5)
- added U43: MCP6002-xMC, Package_DFN_QFN:DFN-8-1EP_3x2mm_P0.5mm_EP1.75x1.45mm, B.Cu at (63.9, 106.0)
- added U44: MCP6002-xMC, Package_DFN_QFN:DFN-8-1EP_3x2mm_P0.5mm_EP1.75x1.45mm, B.Cu at (196.6, 63.2)
- added U45: CD74HC4067M, Package_SO:SOIC-24W_7.5x15.4mm_P1.27mm, B.Cu at (73.6, 107.9)
- added U46: CD74HC4067M, Package_SO:SOIC-24W_7.5x15.4mm_P1.27mm, B.Cu at (206.2, 64.9)
- added U47: MCP6002-xMC, Package_DFN_QFN:DFN-8-1EP_3x2mm_P0.5mm_EP1.75x1.45mm, B.Cu at (197.3, 105.8)
- added U48: CD74HC4067M, Package_SO:SOIC-24W_7.5x15.4mm_P1.27mm, B.Cu at (206.9, 107.4)
- added U5: TMC2209-LA, Package_DFN_QFN:VQFN-28-1EP_5x5mm_P0.5mm_EP3.7x3.7mm_ThermalVias, B.Cu at (61.5, 85.5)
- added U6: TMC2209-LA, Package_DFN_QFN:VQFN-28-1EP_5x5mm_P0.5mm_EP3.7x3.7mm_ThermalVias, B.Cu at (61.8, 94.7)
- added U7: DRV5055A3xDBZxQ1, Package_TO_SOT_SMD:SOT-23, B.Cu at (24.6, 126.4)
- added U8: DRV5055A3xDBZxQ1, Package_TO_SOT_SMD:SOT-23, B.Cu at (43.7, 126.4)
- added U9: DRV5055A3xDBZxQ1, Package_TO_SOT_SMD:SOT-23, B.Cu at (62.7, 126.4)
Other:
- board outline added: 266.7 x 81 mm

Commit message: dc-dc buck converter
Parts:
- removed the REF** at (46.1, 121.3)
- added C81: 4.7μF, Capacitor_SMD:C_0805_2012Metric, B.Cu at (149.5, 87.2)
- added C82: 0.1μF, Capacitor_SMD:C_0805_2012Metric, B.Cu at (143.2, 88.0)
- added C83: 0.1μF, Capacitor_SMD:C_0805_2012Metric, B.Cu at (149.5, 83.8)
- added J8: Conn_01x02_Pin, Connector_PinSocket_2.54mm:PinSocket_1x02_P2.54mm_Vertical, B.Cu at (29.6, 96.0)
- added J9: Conn_01x02_Socket, Connector_PinSocket_2.54mm:PinSocket_1x02_P2.54mm_Vertical, B.Cu at (30.7, 92.3)
- added R26: 10kΩ, Resistor_SMD:R_0805_2012Metric, B.Cu at (135.8, 87.4)
- added R27: 100kΩ, Resistor_SMD:R_0805_2012Metric, B.Cu at (135.8, 83.9)
- added REF**: SW_Cherry_MX_1.00u_PCB_3dmodel, 1_udu_lib:SW_Cherry_MX_1.00u_PCB_3dmodel, F.Cu at (46.1, 121.3)
- added U49: TPS2115APW, 2_udu_lib:PW8, B.Cu at (142.7, 81.8)
- REF** (x35): value SW_Cherry_MX_1.00u_PCB -> SW_Cherry_MX_1.00u_PCB_3dmodel; footprint Button_Switch_Keyboard:SW_Cherry_MX_1.00u_PCB -> 1_udu_lib:SW_Cherry_MX_1.00u_PCB_3dmodel
- REF** (x2): value SW_Cherry_MX_1.00u_PCB -> SW_Cherry_MX_1.00u_PCB_3dmodel_centerhole; footprint Button_Switch_Keyboard:SW_Cherry_MX_1.00u_PCB -> 1_udu_lib:SW_Cherry_MX_1.00u_PCB_3dmodel_centerhole
- TP1: renamed from TP1 TX
- TP2: renamed from TP2 RX
- moved R23 0.50 mm to (135.3, 80.3)
- moved U1 0.24 mm to (138.6, 61.7)
Connections:
- D1 pad 1: +5V -> IN2
Other:
- outline, holes or cut-outs redrawn

Commit message: fix some pcb layout stuff
Routing:
- added copper zone on B.Cu, net (none)
- added copper zone on F.Cu, net GND

Commit message: finish tracing everything
Parts:
- moved C5 117.9 mm to (144.2, 95.7)
- moved C6 117.9 mm to (144.2, 92.2)
- moved U2 117.9 mm to (149.6, 93.9)
- moved J3 35.8 mm to (39.6, 96.0)
- moved J4 33.6 mm to (54.7, 94.2)
- moved J8 22.3 mm to (31.2, 73.8), turned to 90 degrees
- moved C8 21.0 mm to (43.2, 105.0), turned to 0 degrees
- moved J9 20.4 mm to (21.8, 73.9)
- moved J5 19.3 mm to (44.5, 83.9), turned to 180 degrees
- moved C16 18.2 mm to (64.9, 101.5), turned to -90 degrees
- moved R22 18.1 mm to (48.4, 83.8), turned to -90 degrees
- moved C12 17.3 mm to (58.3, 104.0), turned to 0 degrees
- moved R7 16.5 mm to (43.5, 96.0), turned to -90 degrees
- moved U3 15.9 mm to (45.4, 100.9), turned to -90 degrees
- moved C23 14.8 mm to (51.1, 84.3), turned to 0 degrees
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Connections:
- U3 pad 21: Net-(J3-Pin_2) -> Net-(J3-Pin_3)
- U3 pad 26: Net-(J3-Pin_3) -> Net-(J3-Pin_2)
- U4 pad 21: Net-(J4-Pin_2) -> Net-(J4-Pin_3)
- U4 pad 26: Net-(J4-Pin_3) -> Net-(J4-Pin_2)
- U5 pad 21: Net-(J5-Pin_2) -> Net-(J5-Pin_3)
- U5 pad 26: Net-(J5-Pin_3) -> Net-(J5-Pin_2)
- U6 pad 21: Net-(J6-Pin_2) -> Net-(J6-Pin_3)
- U6 pad 26: Net-(J6-Pin_3) -> Net-(J6-Pin_2)
Routing:
- net +3.3V: track 0.00 -> 1056.9 mm, vias 0 -> 12
- net S2: track 0.00 -> 270.2 mm, vias 0 -> 4
- net S3: track 0.00 -> 270.1 mm, vias 0 -> 4
- net S0: track 0.00 -> 251.9 mm, vias 0 -> 5
- net S1: track 0.00 -> 247.1 mm, vias 0 -> 4
- net +24V: track 0.00 -> 191.2 mm, vias 0 -> 12
- net RX: track 0.00 -> 181.7 mm, vias 0 -> 3
- net TX: track 0.00 -> 177.7 mm, vias 0 -> 3
- net Net-(U3-~{PD}/UART): track 0.00 -> 158.5 mm, vias 0 -> 2
- net IN2: track 0.00 -> 141.7 mm, vias 0 -> 4
- net TMC1_STEP: track 0.00 -> 140.7 mm, vias 0 -> 2
- net +5V: track 0.00 -> 140.4 mm
- net TMC1_DIR: track 0.00 -> 139.6 mm, vias 0 -> 2
- net D-: track 0.00 -> 130.2 mm, vias 0 -> 2
- net D+: track 0.00 -> 129.6 mm, vias 0 -> 2
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- added copper zone on B.Cu, net GND
- removed copper zone on B.Cu, net (none)

Commit message: add journal, readme, cad, and assets
Parts:
- added G***: LOGO, 1_udu_lib:stepper_drawing_f, F.Cu at (148.3, 95.4)
- added G***: LOGO, 1_udu_lib:stepper_drawing_b, B.Cu at (147.0, 95.2)
